File: NiclaVCarrier/NiclaVCarrier.kicad_pcb (KiCad board)
At the start: 4 copper layers, 55 x 38 mm, 51 parts, among them CN1 Input, CN2 Output, U1 TPS5430DDA, U2 MAX3485EESA+T, U3 SPX3819M5-L-3-3

Commit message: Updated design
Parts:
- removed the G*** at (134.2, 98.3)
- removed kibuzzard-687D13E0: G***, kibuzzard-687D13E0
- added LD4: Tx, LED_SMD:LED_0603_1608Metric, F.Cu at (147.5, 106.1)
- added LD5: Rx, LED_SMD:LED_0603_1608Metric, F.Cu at (151.0, 106.2)
- added R10: 1k, Resistor_SMD:R_0402_1005Metric, F.Cu at (148.9, 105.6)
- added R11: 1k, Resistor_SMD:R_0402_1005Metric, F.Cu at (152.5, 105.7)
- added R7: 10k, Resistor_SMD:R_0805_2012Metric, F.Cu at (150.8, 93.6)
- added R8: 10k, Resistor_SMD:R_0805_2012Metric, F.Cu at (148.4, 79.9)
- added R9: 10k, Resistor_SMD:R_0805_2012Metric, F.Cu at (148.4, 82.1)
- added kibuzzard-687E9791: G***, kibuzzard-687E9791, F.Cu at (154.7, 105.5)
- added kibuzzard-687E9AA8: G***, kibuzzard-687E9AA8, F.Cu at (149.1, 107.1)
- added kibuzzard-687E9ABC: G***, kibuzzard-687E9ABC, F.Cu at (152.7, 107.2)
- moved R1 8.41 mm to (158.1, 102.5), turned to 180 degrees
- moved kibuzzard-687D1424 4.30 mm to (155.0, 97.3)
Routing:
- net /3V3: track 52.8 -> 74.8 mm
- net /RO: track 14.4 -> 30.3 mm
- net /DI: track 11.5 -> 25.7 mm
- net /B: track 85.7 -> 91.1 mm
- net Net-(JP1-B): track 7.00 -> 3.18 mm
- net Net-(LD5-K): track 0.00 -> 1.78 mm
- net Net-(LD4-K): track 0.00 -> 1.74 mm
- net /DE_RE: track 21.7 -> 20.1 mm, vias 1 -> 2
- net /A: track 94.6 -> 93.3 mm
- net GND: vias 7 -> 59
Other:
- board size 55 x 38 mm -> 64 x 38 mm
