File: NiclaVCarrier/NiclaVCarrier.kicad_sch (KiCad schematic)
At the start: 27 parts, among them CN1 Input, CN2 Output, CN3 I2C, U1 TPS5430DDA, U2 MAX3485EESA+T, U3 SPX3819M5-L-3-3

Commit message: Updated design
Parts:
- added LD4: Tx, LED_SMD:LED_0603_1608Metric, symbol Device:LED
- added LD5: Rx, LED_SMD:LED_0603_1608Metric, symbol Device:LED
- added R10, R11: 1k, Resistor_SMD:R_0402_1005Metric, symbol Device:R
- added R7, R8, R9: 10k, Resistor_SMD:R_0805_2012Metric, symbol Device:R
Connections:
- net 3V3: now also LD4.2 (A), LD5.2 (A), R8.1
- net A: now also R8.2
- net B: now also R9.1
- net DE_RE: now also R7.1
- net DI: now also R11.2
- net GND: now also R7.2, R9.2
- net RO: now also R10.2
- new net: LD5.1 (K), R11.1
- new net: LD4.1 (K), R10.1
Other:
- moved on the sheet: JP1, R1, U2
